File: pcb/mSD-Breakout_v10.brd (EAGLE design)
At the start: 31.8 x 25.4 mm, 17 parts, among them IC1 74LVC244APW, IC2 LDO-TS5204, X1 PASSER, X2 PASSER, X3 PASSER

Commit message: updated schematics
Parts:
- C1, C2, C5, C6: value 1uF -> 2uF
Changed lines of the file:
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@@
 <attribute name="VALUE" x="17.78" y="7.9375" size="0.8128" layer="27" font="vector" ratio="10" rot="R90"/>
 </element>
-<element name="C2" library="rcl" package="C0603" value="1uF" x="24.60625" y="6.19125" smashed="yes" rot="R270">
+<element name="C2" library="rcl" package="C0603" value="2uF" x="24.60625" y="6.19125" smashed="yes" rot="R270">
 <attribute name="NAME" x="23.97125" y="3.81" size="0.8128" layer="27" font="vector" ratio="10"/>
 <attribute name="VALUE" x="24.28875" y="3.65125" size="0.8128" layer="27" font="vector" ratio="10" rot="R270"/>
 </element>
-<element name="C5" library="rcl" package="C0603" value="1uF" x="19.52625" y="6.19125" smashed="yes" rot="R270">
+<element name="C5" library="rcl" package="C0603" value="2uF" x="19.52625" y="6.19125" smashed="yes" rot="R270">
 <attribute name="NAME" x="18.89125" y="3.81" size="0.8128" layer="27" font="vector" ratio="10"/>
 <attribute name="VALUE" x="19.20875" y="3.65125" size="0.8128" layer="27" font="vector" ratio="10" rot="R270"/>
@@
 <attribute name="VALUE" x="9.04875" y="3.4925" size="0.8128" layer="27" font="vector" rot="R270"/>
 </element>
-<element name="C6" library="rcl" package="C0603" value="1uF" x="17.62125" y="6.19125" smashed="yes" rot="R270">
+<element name="C6" library="rcl" package="C0603" value="2uF" x="17.62125" y="6.19125" smashed="yes" rot="R270">
 <attribute name="NAME" x="16.98625" y="3.81" size="0.8128" layer="27" font="vector" ratio="10"/>
 <attribute name="VALUE" x="17.30375" y="3.65125" size="0.8128" layer="27" font="vector" ratio="10" rot="R270"/>
 </element>
-<element name="C1" library="rcl" package="C0603" value="1uF" x="26.51125" y="6.19125" smashed="yes" rot="R270">
+<element name="C1" library="rcl" package="C0603" value="2uF" x="26.51125" y="6.19125" smashed="yes" rot="R270">
 <attribute name="NAME" x="25.87625" y="3.81" size="0.8128" layer="27" font="vector" ratio="10"/>
 <attribute name="VALUE" x="26.19375" y="3.65125" size="0.8128" layer="27" font="vector" ratio="10" rot="R270"/>

Commit message: updated schematic and layout files
Parts:
- IC2: value LDO-TS5204 -> LDO-TS5204-3V3
Changed lines of the file:
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@@
 <?xml version="1.0" encoding="utf-8"?>
 <!DOCTYPE eagle SYSTEM "eagle.dtd">
-<eagle version="6.5.0">
+<eagle version="6.6.0">
 <drawing>
 <settings>
@@
 <attribute name="DIGIKEY" value="WM9750TR-ND" x="1.74625" y="13.6525" size="1.778" layer="27" rot="R270" display="off"/>
 </element>
-<element name="IC2" library="we-power" package="SOT23" value="LDO-TS5204" x="22.06625" y="8.73125" smashed="yes">
+<element name="IC2" library="we-power" package="SOT23" value="LDO-TS5204-3V3" x="22.06625" y="8.73125" smashed="yes">
 <attribute name="NAME" x="21.11375" y="5.55625" size="0.8128" layer="27" font="vector" ratio="10"/>
 <attribute name="VALUE" x="18.25625" y="10.795" size="0.8128" layer="27" font="vector" ratio="10"/>
