File: pcb/mSD-Breakout_v10.sch (EAGLE design)
At the start: 17 parts, among them IC1 74LVC244APW, IC2 LDO-TS5204-3V3, X1 PASSER, X2 PASSER, X3 PASSER

Commit message: cleaned up schematics and layout
Changed lines of the file:
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@@
 <setting verticaltext="up"/>
 </settings>
-<grid distance="0.1" unitdist="inch" unit="inch" style="lines" multiple="1" display="no" altdistance="0.01" altunitdist="inch" altunit="inch"/>
+<grid distance="0.05" unitdist="inch" unit="inch" style="lines" multiple="1" display="yes" altdistance="0.025" altunitdist="inch" altunit="inch"/>
 <layers>
 <layer number="1" name="Top" color="4" fill="1" visible="no" active="no"/>
@@
 <part name="C4" library="rcl" deviceset="C-EU" device="C0603" value="100nF"/>
 <part name="C2" library="rcl" deviceset="C-EU" device="C0603" value="2uF"/>
-<part name="FRAME1" library="frames" deviceset="A4L-LOC" device=""/>
 <part name="+3V4" library="supply1" deviceset="+3V3" device=""/>
 <part name="C5" library="rcl" deviceset="C-EU" device="C0603" value="2uF"/>
@@
 <part name="+3V1" library="supply1" deviceset="+3V3" device=""/>
 <part name="GND1" library="supply1" deviceset="GND" device=""/>
+<part name="FRAME1" library="we-symbol" deviceset="FRAME-A4L" device=""/>
 </parts>
 <sheets>
 <sheet>
 <plain>
-<text x="161.29" y="31.75" size="1.27" layer="95">Released under the Creative Commons Attribution Share-Alike License</text>
-<text x="161.29" y="29.21" size="1.27" layer="95">http://creativecommons.org/licenses/by-sa/4.0/</text>
-<text x="161.29" y="25.4" size="1.27" layer="95">Designed by Andreas Watterott (Watterott electronic)</text>
+<text x="162.56" y="21.59" size="1.27" layer="95">Released under the Creative Commons Attribution Share-Alike License</text>
+<text x="162.56" y="19.05" size="1.27" layer="95">http://creativecommons.org/licenses/by-sa/4.0/</text>
+<text x="162.56" y="15.24" size="1.27" layer="95">Designed by Andreas Watterott (Watterott electronic)</text>
 <text x="152.4" y="68.58" size="1.778" layer="97">Card inserted: CD shorted to GND</text>
 <text x="152.4" y="66.04" size="1.778" layer="97">No Card: CD open</text>
@@
 <attribute name="NAME" x="82.296" y="14.732" size="1.778" layer="95" rot="R180"/>
 <attribute name="VALUE" x="80.645" y="10.033" size="1.778" layer="96"/>
-</instance>
-<instance part="FRAME1" gate="G$1" x="0" y="0" smashed="yes">
-<attribute name="DRAWING_NAME" x="217.17" y="15.24" size="2.54" layer="94" font="vector"/>
-<attribute name="LAST_DATE_TIME" x="217.17" y="10.16" size="2.286" layer="94" font="vector"/>
-<attribute name="SHEET" x="230.505" y="5.08" size="2.54" layer="94" font="vector"/>
 </instance>
 <instance part="+3V4" gate="G$1" x="133.35" y="20.32" smashed="yes" rot="R270">
@@
 <attribute name="VALUE" x="92.71" y="104.14" size="1.778" layer="96" rot="R270"/>
 </instance>
-<instance part="X1" gate="G$1" x="167.64" y="17.78"/>
-<instance part="X2" gate="G$1" x="173.99" y="17.78"/>
-<instance part="X3" gate="G$1" x="180.34" y="17.78"/>
-<instance part="LOGO1" gate="G$1" x="205.74" y="17.78"/>
-<instance part="LOGO2" gate="G$1" x="191.77" y="17.78"/>
+<instance part="X1" gate="G$1" x="165.1" y="7.62"/>
+<instance part="X2" gate="G$1" x="170.18" y="7.62"/>
+<instance part="X3" gate="G$1" x="175.26" y="7.62"/>
+<instance part="LOGO1" gate="G$1" x="198.12" y="7.62"/>
+<instance part="LOGO2" gate="G$1" x="208.28" y="7.62"/>
 <instance part="R1" gate="G$1" x="139.7" y="130.81" smashed="yes" rot="R270">
 <attribute name="NAME" x="141.1986" y="132.08" size="1.778" layer="95" rot="R270"/>
@@
 <attribute name="VALUE" x="92.71" y="82.55" size="1.778" layer="96" rot="R270"/>
 </instance>
+<instance part="FRAME1" gate="G$1" x="0" y="0"/>
 </instances>
 <busses>
